File: Hw_Transmitter/transmitter/transmitter.kicad_pcb (KiCad board)
At the start: 2 copper layers, 98 x 68 mm, 18 parts, among them SW1 SW_SPDT, SW2 toggle switch, U1 BP, U2 nRF24L01+, U3 left joystick, U4 right joystick, U6 ams1117, U7 left joystick mounting, U8 right joystick mounting

Commit message: 1. transmitter: replace ams1117-3.3V with ams1117-5V. 2. remove backup files and update git ignore file.
Parts:
- U6: value ams1117 -> ams1117 - 5V
Connections:
- U1 pad 5V: unconnected-(U1-Pad5V) -> +5V
- U6 pad 1: +3V3 -> +5V
Routing:
- net +5V: track 0.00 -> 29.1 mm
- net +3V3: track 149.4 -> 120.8 mm, vias 6 -> 4
Other:
- board text added: "5V"
Changed lines of the file:
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@@
 	(net 33 "unconnected-(U1-PadPB10)")
 	(net 34 "unconnected-(U1-PadPB13)")
-	(net 35 "unconnected-(U1-Pad5V)")
+	(net 35 "+5V")
 	(net 36 "MOSI")
 	(net 37 "+8V")
@@
 		(tags "Resistor Axial_DIN0207 series Axial Horizontal pin pitch 10.16mm 0.25W = 1/4W length 6.3mm diameter 2.5mm")
 		(property "Reference" "R1"
-			(at 4.88 -2.7 360)
+			(at 4.88 -2.7 0)
 			(layer "F.SilkS")
 			(effects
@@
 		)
 		(property "Value" "20K"
-			(at 5 2 360)
+			(at 5 2 0)
 			(layer "F.Fab")
 			(effects
@@
 		)
 		(fp_text user "${REFERENCE}"
-			(at 5.08 0 360)
+			(at 5.08 0 0)
 			(layer "F.Fab")
 			(effects
@@
 		(tags "Resistor Axial_DIN0207 series Axial Horizontal pin pitch 10.16mm 0.25W = 1/4W length 6.3mm diameter 2.5mm")
 		(property "Reference" "R3"
-			(at 5.08 -2.37 360)
+			(at 5.08 -2.37 0)
 			(layer "F.SilkS")
 			(effects
@@
 		)
 		(property "Value" "100R"
-			(at 5.08 2.37 360)
+			(at 5.08 2.37 0)
 			(layer "F.Fab")
 			(effects
@@
 		)
 		(fp_text user "${REFERENCE}"
-			(at 5.08 0 360)
+			(at 5.08 0 0)
 			(layer "F.Fab")
 			(effects
@@
 		(tags "Resistor Axial_DIN0207 series Axial Horizontal pin pitch 10.16mm 0.25W = 1/4W length 6.3mm diameter 2.5mm")
 		(property "Reference" "R2"
-			(at 5.18 -2.4 360)
+			(at 5.18 -2.4 0)
 			(layer "F.SilkS")
 			(effects
@@
 		)
 		(property "Value" "10K"
-			(at 5.08 2.37 360)
+			(at 5.08 2.37 0)
 			(layer "F.Fab")
 			(effects
@@
 		)
 		(fp_text user "${REFERENCE}"
-			(at 5.08 0 360)
+			(at 5.08 0 0)
 			(layer "F.Fab")
 			(effects
@@
 			)
 		)
-		(property "Value" "ams1117"
+		(property "Value" "ams1117 - 5V"
 			(at 1 -3.3 0)
 			(unlocked yes)
@@
 			(layers "*.Cu" "*.Mask")
 			(remove_unused_layers no)
-			(net 4 "+3V3")
+			(net 35 "+5V")
 			(pinfunction "Vout")
 			(pintype "power_out")
@@
 		(tags "Through hole pin header THT 1x05 2.54mm single row")
 		(property "Reference" "U3"
-			(at 0 -2.33 270)
+			(at 0 -2.33 -90)
 			(layer "F.SilkS")
 			(hide yes)
@@
 		)
 		(fp_text user "${REFERENCE}"
-			(at 0 5.08 360)
+			(at 0 5.08 0)
 			(layer "F.Fab")
 			(effects
@@
 			(layers "*.Cu" "*.Mask")
 			(remove_unused_layers no)
-			(net 35 "unconnected-(U1-Pad5V)")
+			(net 35 "+5V")
 			(pinfunction "5V")
-			(pintype "power_out+no_connect")
+			(pintype "power_out")
 		)
 		(pad "G" thru_hole circle
@@
 		(layer "User.2")
 	)
-	(gr_text "3V3"
+	(gr_text "5V"
 		(at 124.2 112.4 0)
 		(layer "F.SilkS")
@@
 	)
 	(segment
-		(start 134.1 106.9)
-		(end 134.1 85.8)
-		(width 0.5)
-		(layer "F.Cu")
-		(net 4)
-	)
-	(segment
-		(start 129.07 112.07)
-		(end 135.1 118.1)
-		(width 0.5)
-		(layer "F.Cu")
-		(net 4)
-	)
-	(segment
 		(start 160.3 71.3)
 		(end 160.3 72.38)
@@
 	)
 	(segment
-		(start 129.27 111.73)
-		(end 129.07 111.73)
-		(width 0.5)
-		(layer "F.Cu")
-		(net 4)
-	)
-	(segment
-		(start 152.188 123.868)
-		(end 153.4 125.08)
-		(width 0.5)
-		(layer "F.Cu")
-		(net 4)
-	)
-	(segment
-		(start 135.1 118.1)
-		(end 135.1 119.3)
-		(width 0.5)
-		(layer "F.Cu")
-		(net 4)
-	)
-	(segment
 		(start 142.1 85.84)
 		(end 138.16 81.9)
@@
 	)
 	(segment
-		(start 136.668 123.868)
-		(end 152.188 123.868)
-		(width 0.5)
-		(layer "F.Cu")
-		(net 4)
-	)
-	(segment
 		(start 160.92 118.4)
 		(end 164.06 118.4)
@@
 	)
 	(segment
-		(start 134.26 85.8)
-		(end 138.16 81.9)
-		(width 0.5)
-		(layer "F.Cu")
-		(net 4)
-	)
-	(segment
 		(start 160.08 118.4)
 		(end 160.92 118.4)
@@
 	)
 	(segment
-		(start 135.7 122.9)
-		(end 136.668 123.868)
-		(width 0.5)
-		(layer "F.Cu")
-		(net 4)
-	)
-	(segment
 		(start 153.4 81.9)
 		(end 153.6 81.7)
@@
 	)
 	(segment
-		(start 129.07 111.73)
-		(end 129.07 112.07)
-		(width 0.5)
-		(layer "F.Cu")
-		(net 4)
-	)
-	(segment
 		(start 142.1 94.7)
 		(end 142.1 85.84)
@@
 	)
 	(segment
-		(start 134.1 106.9)
-		(end 129.27 111.73)
-		(width 0.5)
-		(layer "F.Cu")
-		(net 4)
-	)
-	(segment
 		(start 142.22 97.02)
 		(end 142.2 97)
@@
 		(net 4)
 	)
-	(segment
-		(start 134.1 85.8)
-		(end 134.26 85.8)
-		(width 0.5)
-		(layer "F.Cu")
-		(net 4)
-	)
-	(via
-		(at 135.7 122.9)
-		(size 0.7)
-		(drill 0.3)
-		(layers "F.Cu" "B.Cu")
-		(net 4)
-	)
 	(via
 		(at 142.1 94.7)
@@
 	)
 	(via
-		(at 135.1 119.3)
-		(size 0.7)
-		(drill 0.3)
-		(layers "F.Cu" "B.Cu")
-		(net 4)
-	)
-	(via
 		(at 142.2 97)
 		(size 0.7)
@@
 	)
 	(segment
+		(start 156 99.54)
+		(end 169.46 113)
+		(width 0.5)
+		(layer "B.Cu")
+		(net 4)
+	)
+	(segment
 		(start 142.2 97)
 		(end 142.2 96.5)
@@
 	)
 	(segment
-		(start 158.3 71.3)
-		(end 160.3 71.3)
+		(start 156 84.5)
+		(end 156 99.54)
 		(width 0.5)
 		(layer "B.Cu")
@@
 	)
 	(segment
-		(start 142.2 96.5)
-		(end 142.1 96.4)
+		(start 153.4 81.9)
+		(end 156 84.5)
 		(width 0.5)
 		(layer "B.Cu")
@@
 	)
 	(segment
-		(start 135.1 122.3)
-		(end 135.7 122.9)
+		(start 158.3 71.3)
+		(end 160.3 71.3)
 		(width 0.5)
 		(layer "B.Cu")
@@
 	)
 	(segment
-		(start 135.1 119.3)
-		(end 135.1 122.3)
+		(start 142.2 96.5)
+		(end 142.1 96.4)
 		(width 0.5)
 		(layer "B.Cu")
@@
 	)
 	(segment
+		(start 134.3 104.3)
+		(end 134.3 90.84)
+		(width 0.5)
+		(layer "F.Cu")
+		(net 35)
+	)
+	(segment
+		(start 129.07 109.53)
+		(end 134.3 104.3)
+		(width 0.5)
+		(layer "F.Cu")
+		(net 35)
+	)
+	(segment
+		(start 134.3 90.84)
+		(end 138.16 86.98)
+		(width 0.5)
+		(layer "F.Cu")
+		(net 35)
+	)
+	(segment
+		(start 129.27 111.73)
+		(end 129.07 111.73)
+		(width 0.5)
+		(layer "F.Cu")
+		(net 35)
+	)
+	(segment
+		(start 129.07 111.73)
+		(end 129.07 112.07)
+		(width 0.5)
+		(layer "F.Cu")
+		(net 35)
+	)
+	(segment
+		(start 129.07 111.73)
+		(end 129.07 109.53)
+		(width 0.5)
+		(layer "F.Cu")
+		(net 35)
+	)
+	(segment
